Commit message: simscape

File: ur5bh/ur5bh1.urdf (robot description, URDF)
Before this commit: robot ur5bh, 21 links, 20 joints
Links:
- link bh_base_link: geometry collision mesh filename=package://bhand_description/meshes/palm_282.stl; visual mesh filename=package://bhand_description/meshes/palm_282.stl
- link bh_finger_11_link: geometry collision mesh filename=package://bhand_description/meshes/knuckle.stl; visual mesh filename=package://bhand_description/meshes/knuckle.stl
- link bh_finger_12_link: geometry collision mesh filename=package://bhand_description/meshes/finger.stl; visual mesh filename=package://bhand_description/meshes/finger.stl
- link bh_finger_13_link: geometry collision mesh filename=package://bhand_description/meshes/finger_tip.stl; visual mesh filename=package://bhand_description/meshes/finger_tip.stl
- link bh_finger_21_link: geometry collision mesh filename=package://bhand_description/meshes/knuckle.stl; visual mesh filename=package://bhand_description/meshes/knuckle.stl
- link bh_finger_22_link: geometry collision mesh filename=package://bhand_description/meshes/finger.stl; visual mesh filename=package://bhand_description/meshes/finger.stl
- link bh_finger_23_link: geometry collision mesh filename=package://bhand_description/meshes/finger_tip.stl; visual mesh filename=package://bhand_description/meshes/finger_tip.stl
- link bh_finger_31_link: geometry collision mesh filename=package://bhand_description/meshes/knuckle_fixed.stl; visual mesh filename=package://bhand_description/meshes/knuckle_fixed.stl
- link bh_finger_32_link: geometry collision mesh filename=package://bhand_description/meshes/finger.stl; visual mesh filename=package://bhand_description/meshes/finger.stl
- link bh_finger_33_link: geometry collision mesh filename=package://bhand_description/meshes/finger_tip.stl; visual mesh filename=package://bhand_description/meshes/finger_tip.stl
