Commit message: urdf02

File: ur5bh_save/ur5bh.urdf (robot description, URDF)
Before this commit: robot ur5bh, 21 links, 20 joints
Links:
- link base_link: geometry collision mesh filename=package://ur_description/meshes/ur5/collision/base.stl; visual mesh filename=package://ur_description/meshes/ur5/visual/base.dae
- link bh_base_link: geometry collision mesh filename=package://bhand_description/meshes/palm_282.dae; visual mesh filename=package://bhand_description/meshes/palm_282.dae
- link bh_finger_11_link: geometry collision mesh filename=package://bhand_description/meshes/knuckle.dae; visual mesh filename=package://bhand_description/meshes/knuckle.dae
- link bh_finger_12_link: geometry collision mesh filename=package://bhand_description/meshes/finger.dae; visual mesh filename=package://bhand_description/meshes/finger.dae
- link bh_finger_13_link: geometry collision mesh filename=package://bhand_description/meshes/finger_tip.dae; visual mesh filename=package://bhand_description/meshes/finger_tip.dae
- link bh_finger_21_link: geometry collision mesh filename=package://bhand_description/meshes/knuckle.dae; visual mesh filename=package://bhand_description/meshes/knuckle.dae
- link bh_finger_22_link: geometry collision mesh filename=package://bhand_description/meshes/finger.dae; visual mesh filename=package://bhand_description/meshes/finger.dae
- link bh_finger_23_link: geometry collision mesh filename=package://bhand_description/meshes/finger_tip.dae; visual mesh filename=package://bhand_description/meshes/finger_tip.dae
- link bh_finger_31_link: geometry collision mesh filename=package://bhand_description/meshes/knuckle_fixed.dae; visual mesh filename=package://bhand_description/meshes/knuckle_fixed.dae
- link bh_finger_32_link: geometry collision mesh filename=package://bhand_description/meshes/finger.dae; visual mesh filename=package://bhand_description/meshes/finger.dae
- link bh_finger_33_link: geometry collision mesh filename=package://bhand_description/meshes/finger_tip.dae; visual mesh filename=package://bhand_description/meshes/finger_tip.dae
- link forearm_link: geometry collision mesh filename=package://ur_description/meshes/ur5/collision/forearm.stl; visual mesh filename=package://ur_description/meshes/ur5/visual/forearm.dae
- link shoulder_link: geometry collision mesh filename=package://ur_description/meshes/ur5/collision/shoulder.stl; visual mesh filename=package://ur_description/meshes/ur5/visual/shoulder.dae
- link upper_arm_link: geometry collision mesh filename=package://ur_description/meshes/ur5/collision/upperarm.stl; visual mesh filename=package://ur_description/meshes/ur5/visual/upperarm.dae
- link wrist_1_link: geometry collision mesh filename=package://ur_description/meshes/ur5/collision/wrist1.stl; visual mesh filename=package://ur_description/meshes/ur5/visual/wrist1.dae
- link wrist_2_link: geometry collision mesh filename=package://ur_description/meshes/ur5/collision/wrist2.stl; visual mesh filename=package://ur_description/meshes/ur5/visual/wrist2.dae
- link wrist_3_link: geometry collision mesh filename=package://ur_description/meshes/ur5/collision/wrist3.stl; visual mesh filename=package://ur_description/meshes/ur5/visual/wrist3.dae
